Commit message: new

File: diff_bot/urdf/caster_wheel.xacro (robot description, xacro)
@@ -16,5 +16,5 @@
             </geometry>
         </collision>
-        <xacro:inertial_sphere mass="${caster_wheel_mass}" radius="${caster_wheel_radius}">
+        <xacro:inertial_sphere mass="${8*caster_wheel_mass}" radius="${2*caster_wheel_radius}">
             <origin xyz="0.0 0.0 0.0" rpy="0.0 0.0 0.0"/>
         </xacro:inertial_sphere>

File: diff_bot/urdf/chassis.xacro (robot description, xacro)
@@ -8,10 +8,10 @@
             </geometry>
             <origin xyz="${chassis_length/2} 0.0 ${chassis_height/2}"/>
-            <material name="green"/>
+            <material name="red"/>
         </visual>
         <collision>
             <origin xyz="${chassis_length/2} 0.0 ${chassis_height/2}"/>
         </collision>
-        <xacro:inertial_box mass="${chassis_mass}" x="${chassis_length}" y="${chassis_width}" z="${chassis_height}">
+        <xacro:inertial_box mass="${chassis_mass}" x="${3*chassis_length}" y="${3*chassis_width}" z="${3*chassis_height}">
             <origin xyz="${chassis_length/2} 0 ${chassis_height/2}" rpy="0 0 0"/>
         </xacro:inertial_box>
@@ -24,5 +24,5 @@
     </joint>
     <gazebo reference="chassis_link">
-        <material> Gazebo/Grey </material>
+        <material> Gazebo/Silver </material>
     </gazebo>
 </robot>

File: diff_bot/urdf/lidar.xacro (robot description, xacro)
@@ -5,5 +5,5 @@
         <visual>
             <geometry>
-                <cylinder radius="0.05" length="0.04"/>
+                <cylinder radius="0.05" length="0.03"/>
             </geometry>
             <material name="black"/>
@@ -16,7 +16,34 @@
     </gazebo>
     <joint name="laser_joint" type="fixed">
-        <origin xyz="0.07 0.0 0.18" rpy="0.0 0.0 0.0"/>
+        <origin xyz="0.07 0.0 0.1" rpy="0.0 0.0 0.0"/>
         <parent link="chassis_link"/>
         <child link="laser_frame"/>
+    </joint>
+       <!-- Caster Holder (Only for visuals) -->
+       <link name="lidar_holder">
+        <visual>
+            <geometry>
+                <cylinder radius="${caster_wheel_radius/2}" length="${caster_wheel_offset_z*2}"/>
+            </geometry>
+            <material name="red"/>
+        </visual>
+    </link>
+    <joint name="lidar_holder_joint" type="fixed">
+        <origin xyz="0.1 0.0 0.07" rpy="0.0 0.0 0.0"/>
+        <parent link="chassis_link"/>
+        <child link="lidar_holder"/>
+    </joint>
+    <link name="lidar_holder2">
+        <visual>
+            <geometry>
+                <cylinder radius="${caster_wheel_radius/2}" length="${caster_wheel_offset_z*2}"/>
+            </geometry>
+            <material name="red"/>
+        </visual>
+    </link>
+    <joint name="lidar_holder_joint2" type="fixed">
+        <origin xyz="0.04 0.0 0.07" rpy="0.0 0.0 0.0"/>
+        <parent link="chassis_link"/>
+        <child link="lidar_holder2"/>
     </joint>
     <!-- Lidar Plugin -->

File: diff_bot/urdf/properties.xacro (robot description, xacro)
@@ -5,5 +5,5 @@
     <xacro:property name="chassis_length" value="0.18"/>
     <xacro:property name="chassis_width" value="0.18"/>
-    <xacro:property name="chassis_height" value="0.11"/>
+    <xacro:property name="chassis_height" value="0.05"/>
     <xacro:property name="chassis_mass" value="1.0"/>
     <!-- Wheels -->
@@ -12,5 +12,5 @@
     <xacro:property name="wheel_offset_z" value="-0.025"/>
     <xacro:property name="wheel_thickness" value="0.027"/>
-    <xacro:property name="wheel_radius" value="0.0325"/>
+    <xacro:property name="wheel_radius" value="0.03"/>
     <xacro:property name="wheel_mass" value="0.037"/>
     <!-- Caster Wheel -->
@@ -18,5 +18,5 @@
     <xacro:property name="caster_wheel_mass" value="0.01"/>
     <xacro:property name="caster_wheel_offset_x" value="0.150"/>
-    <xacro:property name="caster_wheel_offset_z" value="-0.035"/>
+    <xacro:property name="caster_wheel_offset_z" value="-0.025"/>
                                 <!-- Colors -->
     <material name="white">
@@ -24,11 +24,11 @@
     </material>
     <material name="red">
-        <color rgba="1 0 0 1"/>
+        <color rgba="0.5 0.5 0.5 1"/>
     </material>
     <material name="green">
-        <color rgba="0 1 0 1"/>
+        <color rgba="0 0 0 1"/>
     </material>
     <material name="blue">
-        <color rgba="0 0 1 1"/>
+        <color rgba="1 1 1 1"/>
     </material>
     <material name="black">

File: diff_bot/urdf/wheels.xacro (robot description, xacro)
@@ -8,5 +8,5 @@
                     <cylinder radius="${wheel_radius}" length="${wheel_thickness}"/>
                 </geometry>
-                <material name="red"/>
+                <material name="green"/>
             </visual>
             <collision>
